Commit message: First commit

File: simple_rover_description/urdf/simple_rover.urdf (robot description, URDF)
Before this commit: robot simple_rover, 5 links, 4 joints
Links:
- added link body_link, mass 135.5; collision box size=1 0.5 0.1; visual box size=1 0.5 0.1
- added link camera_depth_optical_frame
- added link camera_link; visual mesh filename=package://simple_rover_description/meshes/ZED.stl
- added link zed_left_camera_frame
- added link zed_left_camera_optical_frame
- added link zed_right_camera_frame
- added link zed_right_camera_optical_frame
- link base_link: geometry 
- link wheel_left_back_link: mass None -> 1; geometry collision cylinder length=0.1 radius=0.25; visual cylinder length=0.1 radius=0.25
- link wheel_left_front_link: mass None -> 1; geometry collision cylinder length=0.1 radius=0.25; visual cylinder length=0.1 radius=0.25
- link wheel_right_back_link: mass None -> 1; geometry collision cylinder length=0.1 radius=0.25; visual cylinder length=0.1 radius=0.25
- link wheel_right_front_link: mass None -> 1; geometry collision cylinder length=0.1 radius=0.25; visual cylinder length=0.1 radius=0.25
Joints:
- added joint base_joint: type fixed, parent base_link, child body_link
- added joint camera_depth_optical_frame_joint: type fixed, parent camera_link, child camera_depth_optical_frame, origin xyz=0 0 0 rpy=0 0 0
- added joint origin_joint: type fixed, parent base_link, child camera_link, origin xyz=0 0 0 rpy=0 0 0
- added joint zed_left_camera_joint: type fixed, parent camera_link, child zed_left_camera_frame, origin xyz=0 0.06 0 rpy=0 0 0
- added joint zed_left_camera_optical_joint: type fixed, parent zed_left_camera_frame, child zed_left_camera_optical_frame, origin xyz=0 0 0 rpy=-1.57079632679 0.0 -1.57079632679
- added joint zed_right_camera_joint: type fixed, parent camera_link, child zed_right_camera_frame, origin xyz=0 -0.06 0 rpy=0 0 0
- added joint zed_right_camera_optical_joint: type fixed, parent zed_right_camera_frame, child zed_right_camera_optical_frame, origin xyz=0 0 0 rpy=-1.57079632679 0.0 -1.57079632679

File: simple_rover_description/urdf/simple_rover.urdf.xacro (robot description, xacro)
@@ -21,4 +21,14 @@
   <!-- Import all Gazebo-customization elements, including Gazebo colors -->
   <xacro:include filename="$(find simple_rover_description)/urdf/simple_rover.gazebo" />
+  <!-- Import Rviz colors -->
+  <xacro:include filename="$(find simple_rover_description)/urdf/materials.urdf.xacro" />
+  <!-- ZED depth camera -->
+  <xacro:include filename="$(find simple_rover_description)/urdf/sensors/zed/zed.urdf.xacro" />
+  <!--
+  Used for fixing robot to Gazebo 'base_link'
+  Base link cannot have inertia
+  -->
+  <link name="base_link"/>
+  <!-- Generic wheel macro -->
   <xacro:macro name="wheel" params="pos xyz">
     <link name="wheel_${pos}_link">
@@ -38,4 +48,5 @@
           <cylinder length="${wheel_width}" radius="${wheel_radius}"/>
         </geometry>
+        <material name="blue" />
       </visual>
       <collision>
@@ -52,4 +63,5 @@
       <axis xyz="0 0 1" />
     </joint>
+    <!--
     <transmission name="wheel_${pos}_trans">
       <type>transmission_interface/SimpleTransmission</type>
@@ -59,10 +71,11 @@
       <actuator name="wheel_${pos}_motor">
         <mechanicalReduction>1</mechanicalReduction>
-        <!-- hardwareInterface>EffortJointInterface</hardwareInterface -->
       </actuator>
     </transmission>
+    -->
+    <!-- hardwareInterface>EffortJointInterface</hardwareInterface -->
   </xacro:macro>
-  <!-- Links -->
-  <link name="base_link">
+  <!-- Main body -->
+  <link name="body_link">
     <inertial>
       <origin xyz="0 0 0" rpy="0 0 0"/>
@@ -80,4 +93,5 @@
         <box size="${base_depth} ${base_width} ${base_height}" />
       </geometry>
+      <material name="orange" />
     </visual>
     <collision>
@@ -88,4 +102,8 @@
     </collision>
   </link>
+  <joint name="base_joint" type="fixed">
+    <parent link="base_link"/>
+    <child link="body_link"/>
+  </joint>
   <!-- Wheels -->
   <xacro:wheel pos="right_front"
@@ -97,3 +115,5 @@
   <xacro:wheel pos="left_back"
     xyz="${-base_depth * 0.4} ${base_width / 2 + wheel_width / 2} 0" />
+  <!-- ZED camera -->
+  <xacro:zed_camera parent="base_link" xyz="0 0 0.5" rpy="0 0 0" />
 </robot>
